Commit message: Multisense head by itself is working. Need to create the mobile robot base for the head though.

File: src/cylbot_description/robots/cylbot.urdf.xacro (robot description, xacro)
@@ -1,8 +1,3 @@
 <robot xmlns:xacro="http://www.ros.org/wiki/xacro" name="atlas">
-  <xacro:include filename="$(find multisense_sl_description)/urdf/multisense_sl_v3.urdf" />
-  <!-- <joint name="hokuyo_link_joint" type="fixed"> -->
-  <!-- 	<origin rpy="0 0 0" xyz="0 0 0"/> -->
-  <!-- 	<parent link="head"/> -->
-  <!-- 	<child link="hokuyo_link"/> -->
-  <!-- </joint> -->
+  <xacro:include filename="$(find cylbot_description)/urdf/multisense_sl_v3.urdf" />
 </robot>

Commit message: Head is now attached to a base. However, need to make the wheels more realistic.

File: src/cylbot_description/robots/cylbot.urdf.xacro (robot description, xacro)
@@ -1,3 +1,25 @@
 <robot xmlns:xacro="http://www.ros.org/wiki/xacro" name="atlas">
+  <xacro:include filename="$(find cylbot_description)/urdf/cylbot_base.urdf" />
   <xacro:include filename="$(find cylbot_description)/urdf/multisense_sl_v3.urdf" />
+  <link name="head_tilt_link">
+  </link>
+  <link name="head_offset_link">
+  </link>
+  <joint name="head_pan" type="continuous">
+	<parent link="head_pole"/>
+	<child link="head_tilt_link"/>
+	<axis xyz="0 0 1"/>
+	<origin xyz="0 0 0" rpy="0 0 0"/>
+  </joint>
+  <joint name="head_tilt" type="continuous">
+    <parent link="head_tilt_link"/>
+    <child link="head_offset_link"/>
+	<axis xyz="1 0 0"/>
+    <origin xyz="0 0 0" rpy="0 0 0"/>
+  </joint>
+  <joint name="head_offset" type="fixed">
+	<parent link="head_offset_link"/>
+	<child link="head"/>
+	<origin xyz="0 .1 .1" rpy="0 0 1.57075"/>
+  </joint>
 </robot>

Commit message: Head is now on a simple robot base that shows up properly in both Gazebo and RVIZ. Need to add the controllers for the joints though.

File: src/cylbot_description/robots/cylbot.urdf.xacro (robot description, xacro)
@@ -1,25 +1,7 @@
-<robot xmlns:xacro="http://www.ros.org/wiki/xacro" name="atlas">
+<robot xmlns:xacro="http://www.ros.org/wiki/xacro" name="cylbot">
+  <!-- Gazebo-customization elements -->
+  <xacro:include filename="$(find cylbot_description)/urdf/cylbot_base.gazebo"/>
   <xacro:include filename="$(find cylbot_description)/urdf/cylbot_base.urdf" />
   <xacro:include filename="$(find cylbot_description)/urdf/multisense_sl_v3.urdf" />
-  <link name="head_tilt_link">
-  </link>
-  <link name="head_offset_link">
-  </link>
-  <joint name="head_pan" type="continuous">
-	<parent link="head_pole"/>
-	<child link="head_tilt_link"/>
-	<axis xyz="0 0 1"/>
-	<origin xyz="0 0 0" rpy="0 0 0"/>
-  </joint>
-  <joint name="head_tilt" type="continuous">
-    <parent link="head_tilt_link"/>
-    <child link="head_offset_link"/>
-	<axis xyz="1 0 0"/>
-    <origin xyz="0 0 0" rpy="0 0 0"/>
-  </joint>
-  <joint name="head_offset" type="fixed">
-	<parent link="head_offset_link"/>
-	<child link="head"/>
-	<origin xyz="0 .1 .1" rpy="0 0 1.57075"/>
-  </joint>
+  <!--<link name="head"/>-->
 </robot>

File: src/cylbot_description/urdf/cylbot_base.urdf (robot description, URDF)
Before this commit: robot visual, 10 links, 9 joints
Links:
- removed link left_back_wheel
- removed link left_base
- removed link left_front_wheel
- removed link left_leg
- removed link right_back_wheel
- removed link right_base
- removed link right_front_wheel
- removed link right_leg
- added link back_caster; collision sphere radius=.075; visual sphere radius=.075
- added link front_caster; collision sphere radius=.075; visual sphere radius=.075
- added link head_offset_link, mass .1
- added link head_tilt_link, mass .1
- added link left_wheel, mass 1.5; collision cylinder length=.05 radius=.2; visual cylinder length=.05 radius=.2
- added link right_wheel, mass 1.5; collision cylinder length=.05 radius=.2; visual cylinder length=.05 radius=.2
- link base_link: mass None -> 10; geometry collision cylinder length=0.6 radius=0.2; visual cylinder length=0.6 radius=0.2
- link head_pole: mass None -> .1
Joints:
- removed joint base_to_left_leg
- removed joint base_to_right_leg
- removed joint left_back_wheel_joint
- removed joint left_base_joint
- removed joint left_front_wheel_joint
- removed joint right_back_wheel_joint
- removed joint right_base_joint
- removed joint right_front_wheel_joint
- added joint base_back_caster: type fixed, parent base_link, child back_caster, origin xyz=0 -.125 -.325
- added joint base_front_caster: type fixed, parent base_link, child front_caster, origin xyz=0 .125 -.325
- added joint head_offset: type fixed, parent head_offset_link, child head, origin xyz=0 .1 .1 rpy=0 0 1.57075
- added joint head_pan: type continuous, parent head_pole, child head_tilt_link, origin xyz=0 0 0 rpy=0 0 0, axis 0 0 1
- added joint head_tilt: type continuous, parent head_tilt_link, child head_offset_link, origin xyz=0 0 0 rpy=0 0 0, axis 1 0 0
- added joint left_wheel_joint: type continuous, parent base_link, child left_wheel, origin xyz=-.23 0 -.2 rpy=0 1.57075 0, axis 0 0 1
- added joint right_wheel_joint: type continuous, parent base_link, child right_wheel, origin xyz=.23 0 -.2 rpy=0 1.57075 0, axis 0 0 1
