Commit message: Fixed some issues with the pan and tilt joints

File: src/cylbot_description/urdf/cylbot_base.urdf (robot description, URDF)
Before this commit: robot cylbot, 8 links, 8 joints
Links:
- removed link head_offset_link
- link head_tilt_link: mass .1 -> .01
Joints:
- removed joint head_offset
- joint head_pan: origin xyz=0 0 0 rpy=0 0 0 -> xyz=0 0 .127 rpy=0 0 1.57075
- joint head_tilt: axis 1 0 0 -> 0 1 0; child head_offset_link -> head

Commit message: Fixed the caster wheels on the robot

File: src/cylbot_description/urdf/cylbot_base.urdf (robot description, URDF)
Before this commit: robot cylbot, 7 links, 7 joints
Links:
- removed link back_caster
- added link front_caster_holder, mass .01
- link front_caster: mass None -> .1837; geometry collision cylinder length=.05 radius=.07; visual cylinder length=.05 radius=.07
Joints:
- removed joint base_back_caster
- removed joint base_front_caster
- added joint front_caster_x: type continuous, parent front_caster_holder, child front_caster, origin xyz=0 0 0 rpy=0 1.57075 0, axis 1 0 0
- added joint front_caster_z: type continuous, parent base_link, child front_caster_holder, origin xyz=0 .125 -.325, axis 0 0 1
- joint left_wheel_joint: origin xyz=-.23 0 -.2 rpy=0 1.57075 0 -> xyz=-.24 -.2 -.2 rpy=0 -1.57075 0
- joint right_wheel_joint: origin xyz=.23 0 -.2 rpy=0 1.57075 0 -> xyz=.24 -.2 -.2 rpy=0 -1.57075 0
